File: Quadcopter_FCU/Quadcopter_FCU.sch (KiCad schematic (older format))
At the start: 30 parts

Commit message: completed header implementation for PWM
Parts:
- U?: symbol Regulator_Linear:LM2931-3.3_TO220 -> Quadcopter_FCU-rescue:LM2931-3.3_TO220-Regulator_Linear
Changed lines of the file:
@@
 $EndComp
 $Comp
-L Regulator_Linear:LM2931-3.3_TO220 U?
+L Quadcopter_FCU-rescue:LM2931-3.3_TO220-Regulator_Linear U?
 U 1 1 619CB9E6
 P 3800 1800

Commit message: added PWM setting functionality, and power LEDs to schematic
Parts:
- removed J?: Conn_01x10_Male, symbol Connector:Conn_01x10_Male
- removed J?: Conn_01x04_Male, symbol Connector:Conn_01x04_Male
- added J?: Conn_01x12_Male, symbol Connector:Conn_01x12_Male
- added R5: 5.9k, symbol Device:R
- added R5: 2.4k, symbol Device:R
- added XZVG53W-8 (x2): LED, symbol Device:LED
Connections:
- net +3.3VA: now also J?.1 (Pin_1), J?.7 (Pin_7), R5.1
- net +5V: now also R5.1
- net GND: now also U?.6 (INT), J?.2 (Pin_2), J?.8 (Pin_8), XZVG53W-8.1 (K), XZVG53W-8.1 (K)
- new net: R5.2, XZVG53W-8.2 (A) (x2)
Other:
- note added: "ICM-20602 IMU"
- note added: "POWER LEDs\n"
- note removed: "SPI BREAKOUT PINS\n"
- moved on the sheet: J?

Commit message: associated footprints and generated netlist
Parts:
- C1, C10, C11, C12, C2, C3, C4, C5, C6, C7, C8, C9: footprint (none) -> Capacitor_SMD:C_0805_2012Metric
- J1: renamed from J?; footprint (none) -> Connector_PinHeader_2.00mm:PinHeader_1x12_P2.00mm_Horizontal
- J2, J3: renamed from J?; footprint (none) -> Connector_PinHeader_2.00mm:PinHeader_1x04_P2.00mm_Horizontal
- J4, J5, J6, J7, J8: renamed from J?; footprint (none) -> Connector_PinHeader_2.00mm:PinHeader_1x03_P2.00mm_Horizontal
- J9: renamed from J?; footprint (none) -> Connector_PinHeader_2.00mm:PinHeader_1x06_P2.00mm_Horizontal
- L1, L2: renamed from XZVG53W-8; value LED -> XZVG53W-8; footprint (none) -> LED_SMD:LED_0805_2012Metric
- R1, R5: footprint (none) -> Resistor_SMD:R_0805_2012Metric_Pad1.15x1.40mm_HandSolder
- R2, R3, R4: renamed from R?; footprint (none) -> Resistor_SMD:R_0805_2012Metric_Pad1.15x1.40mm_HandSolder
- R6: renamed from R5; footprint (none) -> Resistor_SMD:R_0805_2012Metric_Pad1.15x1.40mm_HandSolder
- SW1: renamed from SW?; footprint (none) -> Button_Switch_SMD:SW_Push_1P1T_NO_CK_KMR2
- gave numbers to parts that had none: 3

Commit message: layed out ratsnest
Connections:
- net SPI1_MISO: now also J1.5 (Pin_5)
- net SPI1_MOSI: now also J1.6 (Pin_6)
- net SPI1_NSS: now also J1.3 (Pin_3)
- net SPI1_SCK: now also J1.4 (Pin_4)
- net SPI2_MISO: now also J1.11 (Pin_11)
- net SPI2_MOSI: now also J1.12 (Pin_12)
- net SPI2_NSS: now also J1.9 (Pin_9)
- net SPI2_SCK: now also J1.10 (Pin_10)
Changed lines of the file:
@@
 Wire Wire Line
 	3150 1650 3150 1800
+Wire Wire Line
+	1150 2300 1300 2300
+Wire Wire Line
+	1300 2400 1150 2400
+Wire Wire Line
+	1150 2500 1300 2500
+Wire Wire Line
+	1150 2600 1300 2600
+Wire Wire Line
+	1150 2900 1300 2900
+Wire Wire Line
+	1150 3000 1300 3000
+Wire Wire Line
+	1150 3100 1300 3100
+Wire Wire Line
+	1150 3200 1300 3200
 $EndSCHEMATC
